File: USB3.kicad_sch (KiCad schematic)
At the start: 10 parts, among them P1 USB_C_Plug, U1 NCP360SNT1G, U2 WE-TVS-82400102

Commit message: added part nums
Parts:
- CR1: lcsc (none) -> C126837
- U1: lcsc (none) -> C233713
- U2: lcsc (none) -> C5180249
Changed lines of the file:
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@@
       (effects (font (size 1.27 1.27) italic) hide)
+    )
+    (property "lcsc" "C126837" (at 246.38 104.14 0)
+      (effects (font (size 1.27 1.27)) hide)
     )
     (pin "1")
@@
       (effects (font (size 1.27 1.27) italic) hide)
     )
+    (property "LCSC" "" (at 172.72 67.31 0)
+      (effects (font (size 1.27 1.27)) hide)
+    )
+    (property "lcsc" "C233713" (at 172.72 67.31 0)
+      (effects (font (size 1.27 1.27)) hide)
+    )
     (pin "1")
     (pin "2")
@@
       (effects (font (size 1.27 1.27)) hide)
     )
+    (property "lcsc" "C5180249" (at 156.21 92.71 0)
+      (effects (font (size 1.27 1.27)) hide)
+    )

Commit message: fixed things
Parts:
- U1: footprint NCP360:TSOP5_3X1P5_ONS -> TSOP5_3X1P5_ONS
Changed lines of the file:
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@@
   (junction (at 102.87 102.87) (diameter 0) (color 0 0 0 0)
   )
+  (junction (at 162.56 66.04) (diameter 0) (color 0 0 0 0)
+  )
   (junction (at 86.36 143.51) (diameter 0) (color 0 0 0 0)
   )
@@
   (junction (at 104.14 105.41) (diameter 0) (color 0 0 0 0)
   )
+  (junction (at 80.01 143.51) (diameter 0) (color 0 0 0 0)
+  )
   (junction (at 110.49 82.55) (diameter 0) (color 0 0 0 0)
+  )
+  (junction (at 105.41 77.47) (diameter 0) (color 0 0 0 0)
   )
   (junction (at 133.35 66.04) (diameter 0) (color 0 0 0 0)
@@
     (stroke (width 0) (type default))
   )
+  (wire (pts (xy 80.01 143.51) (xy 86.36 143.51))
+    (stroke (width 0) (type default))
+  )
   (wire (pts (xy 110.49 85.09) (xy 109.22 85.09))
     (stroke (width 0) (type default))
@@
     (stroke (width 0) (type default))
   )
+  (wire (pts (xy 105.41 77.47) (xy 101.6 77.47))
+    (stroke (width 0) (type default))
+  )
   (wire (pts (xy 133.35 66.04) (xy 133.35 67.31))
     (stroke (width 0) (type default))
@@
     (stroke (width 0) (type default))
   )
-  (wire (pts (xy 78.74 143.51) (xy 86.36 143.51))
+  (wire (pts (xy 78.74 143.51) (xy 80.01 143.51))
     (stroke (width 0) (type default))
   )
@@
     (stroke (width 0) (type default))
   )
-  (wire (pts (xy 133.35 66.04) (xy 176.53 66.04))
+  (wire (pts (xy 133.35 66.04) (xy 162.56 66.04))
     (stroke (width 0) (type default))
   )
@@
     (stroke (width 0) (type default))
   )
+  (wire (pts (xy 162.56 66.04) (xy 176.53 66.04))
+    (stroke (width 0) (type default))
+  )
   (wire (pts (xy 193.04 109.22) (xy 205.74 109.22))
     (stroke (width 0) (type default))
   )
-  (wire (pts (xy 115.57 77.47) (xy 101.6 77.47))
+  (wire (pts (xy 115.57 77.47) (xy 105.41 77.47))
     (stroke (width 0) (type default))
   )
@@
         (path "/cec59c69-8f0d-4d06-8fee-6cd1bb72d09c/2799dde1-a67f-418b-93ec-27396881451b"
           (reference "C1") (unit 1)
+        )
+      )
+    )
+  )
+  (symbol (lib_id "power:PWR_FLAG") (at 162.56 66.04 0) (unit 1)
+    (in_bom yes) (on_board yes) (dnp no) (fields_autoplaced)
+    (property "Reference" "#FLG02" (at 162.56 64.135 0)
+      (effects (font (size 1.27 1.27)) hide)
+    )
+    (property "Value" "PWR_FLAG" (at 162.56 62.23 0)
+      (effects (font (size 1.27 1.27)))
+    )
+    (property "Footprint" "" (at 162.56 66.04 0)
+      (effects (font (size 1.27 1.27)) hide)
+    )
+    (property "Datasheet" "~" (at 162.56 66.04 0)
+      (effects (font (size 1.27 1.27)) hide)
+    )
+    (pin "1")
+    (instances
+      (project "framework_logic_analyzer"
+        (path "/cec59c69-8f0d-4d06-8fee-6cd1bb72d09c/2799dde1-a67f-418b-93ec-27396881451b"
+          (reference "#FLG02") (unit 1)
         )
       )
@@
     )
   )
+  (symbol (lib_id "power:PWR_FLAG") (at 80.01 143.51 180) (unit 1)
+    (in_bom yes) (on_board yes) (dnp no)
+    (property "Reference" "#FLG03" (at 80.01 145.415 0)
+      (effects (font (size 1.27 1.27)) hide)
+    )
+    (property "Value" "PWR_FLAG" (at 77.47 147.32 0)
+      (effects (font (size 1.27 1.27)))
+    )
+    (property "Footprint" "" (at 80.01 143.51 0)
+      (effects (font (size 1.27 1.27)) hide)
+    )
+    (property "Datasheet" "~" (at 80.01 143.51 0)
+      (effects (font (size 1.27 1.27)) hide)
+    )
+    (pin "1")
+    (instances
+      (project "framework_logic_analyzer"
+        (path "/cec59c69-8f0d-4d06-8fee-6cd1bb72d09c/2799dde1-a67f-418b-93ec-27396881451b"
+          (reference "#FLG03") (unit 1)
+        )
+      )
+    )
+  )
+  (symbol (lib_id "power:PWR_FLAG") (at 105.41 77.47 0) (unit 1)
+    (in_bom yes) (on_board yes) (dnp no) (fields_autoplaced)
+    (property "Reference" "#FLG01" (at 105.41 75.565 0)
+      (effects (font (size 1.27 1.27)) hide)
+    )
+    (property "Value" "PWR_FLAG" (at 105.41 73.66 0)
+      (effects (font (size 1.27 1.27)))
+    )
+    (property "Footprint" "" (at 105.41 77.47 0)
+      (effects (font (size 1.27 1.27)) hide)
+    )
+    (property "Datasheet" "~" (at 105.41 77.47 0)
+      (effects (font (size 1.27 1.27)) hide)
+    )
+    (pin "1")
+    (instances
+      (project "framework_logic_analyzer"
+        (path "/cec59c69-8f0d-4d06-8fee-6cd1bb72d09c/2799dde1-a67f-418b-93ec-27396881451b"
+          (reference "#FLG01") (unit 1)
+        )
+      )
+    )
+  )
   (symbol (lib_id "power:VBUS") (at 226.06 64.77 0) (unit 1)
     (in_bom yes) (on_board yes) (dnp no) (fields_autoplaced)
@@
       (effects (font (size 1.524 1.524)))
     )
-    (property "Footprint" "NCP360:TSOP5_3X1P5_ONS" (at 172.72 67.31 0)
+    (property "Footprint" "TSOP5_3X1P5_ONS" (at 172.72 67.31 0)
       (effects (font (size 1.27 1.27) italic) hide)
     )
@@
       (effects (font (size 1.27 1.27)) hide)
     )
-    (pin "1")
     (pin "2")
     (pin "3")
     (pin "4")
+    (pin "1")
     (pin "5")
     (instances
