File: power.kicad_sch (KiCad schematic)
At the start: 7 parts, among them U3 AP2112K-3.3, U4 SC189CSKTRT

Commit message: added part nums
Parts:
- L1: LCSC C315721 -> (none); lcsc (none) -> C315721
- U3: lcsc (none) -> C51118
- U4: lcsc (none) -> C2871822
Changed lines of the file:
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@@
+      (effects (font (size 1.27 1.27)) hide)
+    )
+    (property "lcsc" "C51118" (at 76.2 46.99 0)
       (effects (font (size 1.27 1.27)) hide)
     )
@@
       (effects (font (size 1.27 1.27)) hide)
     )
-    (property "LCSC" "C315721" (at 99.06 92.71 90)
+    (property "LCSC" "" (at 99.06 92.71 90)
+      (effects (font (size 1.27 1.27)) hide)
+    )
+    (property "lcsc" "C315721" (at 99.06 92.71 0)
       (effects (font (size 1.27 1.27)) hide)
     )
@@
       (effects (font (size 1.27 1.27) italic) hide)
     )
-    (pin "1")
+    (property "lcsc" "C2871822" (at 58.42 95.25 0)
+      (effects (font (size 1.27 1.27)) hide)
+    )
+    (pin "1")

Commit message: fixed things
Parts:
- U4: footprint SC189:SOT_CSKTRT_SEM -> SOT_CSKTRT_SEM
Connections:
- net +3V3 renamed +3.3V
Changed lines of the file:
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@@
   (junction (at 63.5 95.25) (diameter 0) (color 0 0 0 0)
   )
-  (junction (at 63.5 44.45) (diameter 0) (color 0 0 0 0)
-  )
   (junction (at 63.5 92.71) (diameter 0) (color 0 0 0 0)
   )
-  (junction (at 87.63 57.15) (diameter 0) (color 0 0 0 0)
-  )
   (junction (at 92.71 57.15) (diameter 0) (color 0 0 0 0)
   )
@@
     (stroke (width 0) (type default))
   )
+  (wire (pts (xy 105.41 104.14) (xy 105.41 107.95))
+    (stroke (width 0) (type default))
+  )
+  (wire (pts (xy 105.41 95.25) (xy 105.41 99.06))
+    (stroke (width 0) (type default))
+  )
+  (wire (pts (xy 63.5 95.25) (xy 63.5 99.06))
+    (stroke (width 0) (type default))
+  )
+  (wire (pts (xy 92.71 57.15) (xy 92.71 58.42))
+    (stroke (width 0) (type default))
+  )
+  (wire (pts (xy 63.5 92.71) (xy 63.5 95.25))
+    (stroke (width 0) (type default))
+  )
+  (wire (pts (xy 68.58 46.99) (xy 66.04 46.99))
+    (stroke (width 0) (type default))
+  )
+  (wire (pts (xy 105.41 107.95) (xy 78.74 107.95))
+    (stroke (width 0) (type default))
+  )
+  (wire (pts (xy 92.71 46.99) (xy 92.71 44.45))
+    (stroke (width 0) (type default))
+  )
+  (wire (pts (xy 58.42 57.15) (xy 76.2 57.15))
+    (stroke (width 0) (type default))
+  )
+  (wire (pts (xy 58.42 44.45) (xy 66.04 44.45))
+    (stroke (width 0) (type default))
+  )
+  (wire (pts (xy 58.42 53.34) (xy 58.42 57.15))
+    (stroke (width 0) (type default))
+  )
+  (wire (pts (xy 96.52 92.71) (xy 93.98 92.71))
+    (stroke (width 0) (type default))
+  )
+  (wire (pts (xy 76.2 57.15) (xy 92.71 57.15))
+    (stroke (width 0) (type default))
+  )
+  (wire (pts (xy 105.41 95.25) (xy 105.41 92.71))
+    (stroke (width 0) (type default))
+  )
+  (wire (pts (xy 92.71 38.1) (xy 92.71 44.45))
+    (stroke (width 0) (type default))
+  )
+  (wire (pts (xy 93.98 95.25) (xy 105.41 95.25))
+    (stroke (width 0) (type default))
+  )
+  (wire (pts (xy 83.82 44.45) (xy 92.71 44.45))
+    (stroke (width 0) (type default))
+  )
+  (wire (pts (xy 63.5 107.95) (xy 63.5 104.14))
+    (stroke (width 0) (type default))
+  )
+  (wire (pts (xy 76.2 54.61) (xy 76.2 57.15))
+    (stroke (width 0) (type default))
+  )
+  (wire (pts (xy 66.04 46.99) (xy 66.04 44.45))
+    (stroke (width 0) (type default))
+  )
+  (wire (pts (xy 101.6 92.71) (xy 105.41 92.71))
+    (stroke (width 0) (type default))
+  )
+  (wire (pts (xy 105.41 90.17) (xy 105.41 92.71))
+    (stroke (width 0) (type default))
+  )
+  (wire (pts (xy 92.71 52.07) (xy 92.71 57.15))
+    (stroke (width 0) (type default))
+  )
+  (wire (pts (xy 63.5 90.17) (xy 63.5 92.71))
+    (stroke (width 0) (type default))
+  )
+  (wire (pts (xy 78.74 107.95) (xy 63.5 107.95))
+    (stroke (width 0) (type default))
+  )
+  (wire (pts (xy 78.74 107.95) (xy 78.74 109.22))
+    (stroke (width 0) (type default))
+  )
   (wire (pts (xy 58.42 38.1) (xy 58.42 44.45))
-    (stroke (width 0) (type default))
-  )
-  (wire (pts (xy 105.41 104.14) (xy 105.41 107.95))
-    (stroke (width 0) (type default))
-  )
-  (wire (pts (xy 92.71 38.1) (xy 92.71 44.45))
-    (stroke (width 0) (type default))
-  )
-  (wire (pts (xy 105.41 95.25) (xy 105.41 99.06))
-    (stroke (width 0) (type default))
-  )
-  (wire (pts (xy 63.5 95.25) (xy 63.5 99.06))
-    (stroke (width 0) (type default))
-  )
-  (wire (pts (xy 92.71 57.15) (xy 92.71 58.42))
-    (stroke (width 0) (type default))
-  )
-  (wire (pts (xy 63.5 92.71) (xy 63.5 95.25))
-    (stroke (width 0) (type default))
-  )
-  (wire (pts (xy 68.58 46.99) (xy 66.04 46.99))
-    (stroke (width 0) (type default))
-  )
-  (wire (pts (xy 105.41 107.95) (xy 78.74 107.95))
-    (stroke (width 0) (type default))
-  )
-  (wire (pts (xy 105.41 90.17) (xy 105.41 92.71))
-    (stroke (width 0) (type default))
-  )
-  (wire (pts (xy 92.71 46.99) (xy 92.71 44.45))
-    (stroke (width 0) (type default))
-  )
-  (wire (pts (xy 58.42 57.15) (xy 76.2 57.15))
-    (stroke (width 0) (type default))
-  )
-  (wire (pts (xy 63.5 44.45) (xy 66.04 44.45))
-    (stroke (width 0) (type default))
-  )
-  (wire (pts (xy 58.42 53.34) (xy 58.42 57.15))
-    (stroke (width 0) (type default))
-  )
-  (wire (pts (xy 96.52 92.71) (xy 93.98 92.71))
-    (stroke (width 0) (type default))
-  )
-  (wire (pts (xy 76.2 57.15) (xy 87.63 57.15))
-    (stroke (width 0) (type default))
-  )
-  (wire (pts (xy 105.41 95.25) (xy 105.41 92.71))
-    (stroke (width 0) (type default))
-  )
-  (wire (pts (xy 93.98 95.25) (xy 105.41 95.25))
-    (stroke (width 0) (type default))
-  )
-  (wire (pts (xy 83.82 44.45) (xy 92.71 44.45))
-    (stroke (width 0) (type default))
-  )
-  (wire (pts (xy 63.5 107.95) (xy 63.5 104.14))
-    (stroke (width 0) (type default))
-  )
-  (wire (pts (xy 58.42 44.45) (xy 63.5 44.45))
-    (stroke (width 0) (type default))
-  )
-  (wire (pts (xy 76.2 54.61) (xy 76.2 57.15))
-    (stroke (width 0) (type default))
-  )
-  (wire (pts (xy 66.04 46.99) (xy 66.04 44.45))
-    (stroke (width 0) (type default))
-  )
-  (wire (pts (xy 101.6 92.71) (xy 105.41 92.71))
-    (stroke (width 0) (type default))
-  )
-  (wire (pts (xy 92.71 52.07) (xy 92.71 57.15))
-    (stroke (width 0) (type default))
-  )
-  (wire (pts (xy 87.63 57.15) (xy 92.71 57.15))
-    (stroke (width 0) (type default))
-  )
-  (wire (pts (xy 63.5 90.17) (xy 63.5 92.71))
-    (stroke (width 0) (type default))
-  )
-  (wire (pts (xy 78.74 107.95) (xy 63.5 107.95))
-    (stroke (width 0) (type default))
-  )
-  (wire (pts (xy 78.74 107.95) (xy 78.74 109.22))
     (stroke (width 0) (type default))
   )
@@
         (path "/fff17096-2243-44cc-8e16-f85582cd0560"
           (reference "U3") (unit 1)
-        )
-      )
-    )
-  )
-  (symbol (lib_id "Microcontroller-rescue:+3.3V-power") (at 92.71 38.1 0) (unit 1)
-    (in_bom yes) (on_board yes) (dnp no)
-    (property "Reference" "#PWR013" (at 92.71 41.91 0)
-      (effects (font (size 1.27 1.27)) hide)
-    )
-    (property "Value" "+3.3V" (at 93.091 33.7058 0)
-      (effects (font (size 1.27 1.27)))
-    )
-    (property "Footprint" "" (at 92.71 38.1 0)
-      (effects (font (size 1.27 1.27)) hide)
-    )
-    (property "Datasheet" "" (at 92.71 38.1 0)
-      (effects (font (size 1.27 1.27)) hide)
-    )
-    (pin "1")
-    (instances
-      (project "framework_logic_analyzer"
-        (path "/cec59c69-8f0d-4d06-8fee-6cd1bb72d09c/df825620-032c-4492-9362-da032e4f40e2"
-          (reference "#PWR013") (unit 1)
-        )
-      )
-      (project "Microcontroller"
-        (path "/fff17096-2243-44cc-8e16-f85582cd0560"
-          (reference "#PWR022") (unit 1)
         )
       )
@@
     )
   )
-  (symbol (lib_id "power:PWR_FLAG") (at 63.5 44.45 0) (unit 1)
-    (in_bom yes) (on_board yes) (dnp no)
-    (property "Reference" "#FLG01" (at 63.5 42.545 0)
-      (effects (font (size 1.27 1.27)) hide)
-    )
-    (property "Value" "PWR_FLAG" (at 63.5 40.0558 0)
-      (effects (font (size 1.27 1.27)))
-    )
-    (property "Footprint" "" (at 63.5 44.45 0)
-      (effects (font (size 1.27 1.27)) hide)
-    )
-    (property "Datasheet" "~" (at 63.5 44.45 0)
-      (effects (font (size 1.27 1.27)) hide)
-    )
-    (pin "1")
-    (instances
-      (project "framework_logic_analyzer"
-        (path "/cec59c69-8f0d-4d06-8fee-6cd1bb72d09c/df825620-032c-4492-9362-da032e4f40e2"
-          (reference "#FLG01") (unit 1)
-        )
-      )
-      (project "Microcontroller"
-        (path "/fff17096-2243-44cc-8e16-f85582cd0560"
-          (reference "#FLG02") (unit 1)
+  (symbol (lib_id "power:+3.3V") (at 92.71 38.1 0) (unit 1)
+    (in_bom yes) (on_board yes) (dnp no) (fields_autoplaced)
+    (property "Reference" "#PWR072" (at 92.71 41.91 0)
+      (effects (font (size 1.27 1.27)) hide)
+    )
+    (property "Value" "+3.3V" (at 92.71 34.29 0)
+      (effects (font (size 1.27 1.27)))
+    )
+    (property "Footprint" "" (at 92.71 38.1 0)
+      (effects (font (size 1.27 1.27)) hide)
+    )
+    (property "Datasheet" "" (at 92.71 38.1 0)
+      (effects (font (size 1.27 1.27)) hide)
+    )
+    (pin "1")
+    (instances
+      (project "framework_logic_analyzer"
+        (path "/cec59c69-8f0d-4d06-8fee-6cd1bb72d09c/df825620-032c-4492-9362-da032e4f40e2"
+          (reference "#PWR072") (unit 1)
         )
       )
@@
       (effects (font (size 1.524 1.524)))
     )
-    (property "Footprint" "SC189:SOT_CSKTRT_SEM" (at 58.42 95.25 0)
+    (property "Footprint" "SOT_CSKTRT_SEM" (at 58.42 95.25 0)
       (effects (font (size 1.27 1.27) italic) hide)
     )
@@
         )
       )
-    )
-  )
-  (symbol (lib_id "power:PWR_FLAG") (at 87.63 57.15 0) (unit 1)
-    (in_bom yes) (on_board yes) (dnp no)
-    (property "Reference" "#FLG02" (at 87.63 55.245 0)
-      (effects (font (size 1.27 1.27)) hide)
-    )
-    (property "Value" "PWR_FLAG" (at 87.63 52.7558 0)
-      (effects (font (size 1.27 1.27)))
-    )
-    (property "Footprint" "" (at 87.63 57.15 0)
-      (effects (font (size 1.27 1.27)) hide)
-    )
-    (property "Datasheet" "~" (at 87.63 57.15 0)
-      (effects (font (size 1.27 1.27)) hide)
-    )
-    (pin "1")
-    (instances
-      (project "framework_logic_analyzer"
-        (path "/cec59c69-8f0d-4d06-8fee-6cd1bb72d09c/df825620-032c-4492-9362-da032e4f40e2"
-          (reference "#FLG02") (unit 1)
-        )
-      )
-      (project "Microcontroller"
-        (path "/fff17096-2243-44cc-8e16-f85582cd0560"
-          (reference "#FLG03") (unit 1)
-        )
-      )
